File: micromouse5/micromouse5.kicad_sch (KiCad schematic)
At the start: 69 parts, among them J1 Conn_01x06_Pin, J2 Conn_01x06_Pin, J3 JST 2, J4 JST 1, J5 Conn_01x04_Pin, Q1 IR Receiver, Q2 IR Receiver, Q3 IR Receiver, Q4 IR Receiver, SW1 Button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

Commit message: PCB start
Parts:
- added Motor1, Motor2: ~, Pololu_Motor:Pololu_Motor, symbol pololu_motor:Pololu_Motor
Changed lines of the file:
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@@
+	)
+	(symbol
+		(lib_id "pololu_motor:Pololu_Motor")
+		(at 172.72 331.47 0)
+		(unit 1)
+		(exclude_from_sim no)
+		(in_bom yes)
+		(on_board yes)
+		(dnp no)
+		(fields_autoplaced yes)
+		(property "Reference" "Motor1"
+			(at 180.34 323.2149 0)
+			(effects
+				(font
+					(size 1.27 1.27)
+				)
+				(justify left)
+			)
+		)
+		(property "Value" "~"
+			(at 180.34 325.12 0)
+			(effects
+				(font
+					(size 1.27 1.27)
+				)
+				(justify left)
+			)
+		)
+		(property "Footprint" "Pololu_Motor:Pololu_Motor"
+			(at 172.72 331.47 0)
+			(effects
+				(font
+					(size 1.27 1.27)
+				)
+				(hide yes)
+			)
+		)
+		(property "Datasheet" ""
+			(at 172.72 331.47 0)
+			(effects
+				(font
+					(size 1.27 1.27)
+				)
+				(hide yes)
+			)
+		)
+		(property "Description" ""
+			(at 172.72 331.47 0)
+			(effects
+				(font
+					(size 1.27 1.27)
+				)
+				(hide yes)
+			)
+		)
+		(instances
+			(project ""
+				(path "/afbe2d40-4a52-44ad-a632-ed06745a7c8a"
+					(reference "Motor1")
+					(unit 1)
+				)
+			)
+		)
 	)
 	(symbol
@@
 					(unit 1)
 				)
+			)
+		)
+	)
+	(symbol
+		(lib_id "pololu_motor:Pololu_Motor")
+		(at 200.66 331.47 0)
+		(unit 1)
+		(exclude_from_sim no)
+		(in_bom yes)
+		(on_board yes)
+		(dnp no)
+		(fields_autoplaced yes)
+		(property "Reference" "Motor2"
+			(at 208.28 323.2149 0)
+			(effects
+				(font
+					(size 1.27 1.27)
+				)
+				(justify left)
+			)
+		)
+		(property "Value" "~"
+			(at 208.28 325.12 0)
+			(effects
+				(font
+					(size 1.27 1.27)
+				)
+				(justify left)
+			)
+		)
+		(property "Footprint" "Pololu_Motor:Pololu_Motor"
+			(at 200.66 331.47 0)
+			(effects
+				(font
+					(size 1.27 1.27)
+				)
+				(hide yes)
+			)
+		)
+		(property "Datasheet" ""
+			(at 200.66 331.47 0)
+			(effects
+				(font
+					(size 1.27 1.27)
+				)
+				(hide yes)
+			)
+		)
+		(property "Description" ""
+			(at 200.66 331.47 0)
+			(effects
+				(font
+					(size 1.27 1.27)
+				)
+				(hide yes)
+			)
+		)
+		(instances
+			(project ""
+				(path "/afbe2d40-4a52-44ad-a632-ed06745a7c8a"
+					(reference "Motor2")
+					(unit 1)
+				)

Commit message: PCB work
Connections:
- net at R2.2, U3.1: now also R3.2
- net at R5.2, U4.1: now also R7.2
- net at R15.2: now also R13.2, U6.1
- net at R11.2: now also R9.2, U5.1
Other:
- moved on the sheet: R13, R2, R5, R9
